File: PCB/Full Keyboard.kicad_pcb (KiCad board)
At the start: 4 copper layers, 38.1 x 57.2 mm, 26 parts, among them J1 USB_C, SW1 SW_Push, U1 STM32F072CBT6, U3 XC6206, U4 USBLC6-2SC6

Commit message: commit during highway call
Parts:
- added "-"1: Keyswitch, ScottoKeebs_Hotswap:Hotswap_MX_1.00u, F.Cu at (236.9, 258.2)
- added "0"1: Keyswitch, ScottoKeebs_Hotswap:Hotswap_MX_1.00u, F.Cu at (217.8, 258.2)
- added "1: Keyswitch, ScottoKeebs_Hotswap:Hotswap_MX_1.00u, F.Cu at (248.8, 296.3)
- added "1"1: Keyswitch, ScottoKeebs_Hotswap:Hotswap_MX_1.00u, F.Cu at (46.4, 258.2)
- added "2"1: Keyswitch, ScottoKeebs_Hotswap:Hotswap_MX_1.00u, F.Cu at (65.4, 258.2)
- added "3"1: Keyswitch, ScottoKeebs_Hotswap:Hotswap_MX_1.00u, F.Cu at (84.5, 258.2)
- added "4"1: Keyswitch, ScottoKeebs_Hotswap:Hotswap_MX_1.00u, F.Cu at (103.5, 258.2)
- added "5"1: Keyswitch, ScottoKeebs_Hotswap:Hotswap_MX_1.00u, F.Cu at (122.6, 258.2)
- added "6"1: Keyswitch, ScottoKeebs_Hotswap:Hotswap_MX_1.00u, F.Cu at (141.6, 258.2)
- added "7"1: Keyswitch, ScottoKeebs_Hotswap:Hotswap_MX_1.00u, F.Cu at (160.7, 258.2)
- added "8"1: Keyswitch, ScottoKeebs_Hotswap:Hotswap_MX_1.00u, F.Cu at (179.7, 258.2)
- added "9"1: Keyswitch, ScottoKeebs_Hotswap:Hotswap_MX_1.00u, F.Cu at (198.8, 258.2)
- added "="1: Keyswitch, ScottoKeebs_Hotswap:Hotswap_MX_1.00u, F.Cu at (255.9, 258.2)
- added "?"1: Keyswitch, ScottoKeebs_Hotswap:Hotswap_MX_1.00u, F.Cu at (-0.47, 31.2)
- added ;1: Keyswitch, ScottoKeebs_Hotswap:Hotswap_MX_1.00u, F.Cu at (229.7, 296.3)
- added <1: Keyswitch, ScottoKeebs_Hotswap:Hotswap_MX_1.00u, F.Cu at (-0.47, 62.3)
- added >1: Keyswitch, ScottoKeebs_Hotswap:Hotswap_MX_1.00u, F.Cu at (-0.47, 77.8)
- added A1: Keyswitch, ScottoKeebs_Hotswap:Hotswap_MX_1.00u, F.Cu at (58.3, 296.3)
- added B1: Keyswitch, ScottoKeebs_Hotswap:Hotswap_MX_1.00u, F.Cu at (-0.47, 108.9)
- added Backspace1: Keyswitch, ScottoKeebs_Hotswap:Hotswap_MX_1.00u, F.Cu at (284.5, 258.2)
- added C1: Keyswitch, ScottoKeebs_Hotswap:Hotswap_MX_1.00u, F.Cu at (-0.47, 140.0)
- added CapsLock1: Keyswitch, ScottoKeebs_Hotswap:Hotswap_MX_1.00u, F.Cu at (34.5, 296.3)
- added D1: Diode, ScottoKeebs_Components:Diode_SOD-123, F.Cu at (126.6, 9.54)
- added D10: Diode, ScottoKeebs_Components:Diode_SOD-123, F.Cu at (126.6, 39.7)
- added D100: Diode, ScottoKeebs_Components:Diode_SOD-123, F.Cu at (166.9, 36.3)
- added D101: Diode, ScottoKeebs_Components:Diode_SOD-123, F.Cu at (166.9, 39.7)
- added D102: Diode, ScottoKeebs_Components:Diode_SOD-123, F.Cu at (166.9, 43.0)
- added D103: Diode, ScottoKeebs_Components:Diode_SOD-123, F.Cu at (166.9, 46.4)
- added D104: Diode, ScottoKeebs_Components:Diode_SOD-123, F.Cu at (166.9, 49.7)
- added D105: Keyswitch, ScottoKeebs_Hotswap:Hotswap_MX_1.00u, F.Cu at (96.4, 296.3)
- added D106: LED_WS2812B, ScottoKeebs_Components:LED_WS2812B, F.Cu at (176.0, 11.2)
- added D107: LED_WS2812B, ScottoKeebs_Components:LED_WS2812B, F.Cu at (176.0, 17.8)
- added D108: LED_WS2812B, ScottoKeebs_Components:LED_WS2812B, F.Cu at (176.0, 24.4)
- added D109: LED_WS2812B, ScottoKeebs_Components:LED_WS2812B, F.Cu at (176.0, 31.0)
- added D11: Diode, ScottoKeebs_Components:Diode_SOD-123, F.Cu at (126.6, 43.0)
- added D110: LED_WS2812B, ScottoKeebs_Components:LED_WS2812B, F.Cu at (176.0, 37.7)
- added D111: LED_WS2812B, ScottoKeebs_Components:LED_WS2812B, F.Cu at (176.0, 44.3)
- added D112: LED_WS2812B, ScottoKeebs_Components:LED_WS2812B, F.Cu at (176.0, 50.9)
- added D113: LED_WS2812B, ScottoKeebs_Components:LED_WS2812B, F.Cu at (176.0, 57.5)
- added D114: LED_WS2812B, ScottoKeebs_Components:LED_WS2812B, F.Cu at (176.0, 64.1)
- added D115: LED_WS2812B, ScottoKeebs_Components:LED_WS2812B, F.Cu at (176.0, 70.8)
- added D116: LED_WS2812B, ScottoKeebs_Components:LED_WS2812B, F.Cu at (176.0, 77.4)
- added D117: LED_WS2812B, ScottoKeebs_Components:LED_WS2812B, F.Cu at (176.0, 84.0)
- added D118: LED_WS2812B, ScottoKeebs_Components:LED_WS2812B, F.Cu at (176.0, 90.6)
- added D119: LED_WS2812B, ScottoKeebs_Components:LED_WS2812B, F.Cu at (176.0, 97.2)
- added D12: Diode, ScottoKeebs_Components:Diode_SOD-123, F.Cu at (126.6, 46.4)
- added D120: LED_WS2812B, ScottoKeebs_Components:LED_WS2812B, F.Cu at (176.0, 103.9)
- added D121: LED_WS2812B, ScottoKeebs_Components:LED_WS2812B, F.Cu at (184.4, 11.2)
- added D122: LED_WS2812B, ScottoKeebs_Components:LED_WS2812B, F.Cu at (184.4, 17.8)
- added D123: LED_WS2812B, ScottoKeebs_Components:LED_WS2812B, F.Cu at (184.4, 24.4)
- added D124: LED_WS2812B, ScottoKeebs_Components:LED_WS2812B, F.Cu at (184.4, 31.0)
- added D125: LED_WS2812B, ScottoKeebs_Components:LED_WS2812B, F.Cu at (184.4, 37.7)
- added D126: LED_WS2812B, ScottoKeebs_Components:LED_WS2812B, F.Cu at (184.4, 44.3)
- added D127: LED_WS2812B, ScottoKeebs_Components:LED_WS2812B, F.Cu at (184.4, 50.9)
- added D128: LED_WS2812B, ScottoKeebs_Components:LED_WS2812B, F.Cu at (184.4, 57.5)
- added D129: LED_WS2812B, ScottoKeebs_Components:LED_WS2812B, F.Cu at (184.4, 64.1)
- added D13: Diode, ScottoKeebs_Components:Diode_SOD-123, F.Cu at (126.6, 49.7)
- added D130: LED_WS2812B, ScottoKeebs_Components:LED_WS2812B, F.Cu at (184.4, 70.8)
- added D131: LED_WS2812B, ScottoKeebs_Components:LED_WS2812B, F.Cu at (184.4, 77.4)
- added D132: LED_WS2812B, ScottoKeebs_Components:LED_WS2812B, F.Cu at (184.4, 84.0)
- added D133: LED_WS2812B, ScottoKeebs_Components:LED_WS2812B, F.Cu at (184.4, 90.6)
- added D134: LED_WS2812B, ScottoKeebs_Components:LED_WS2812B, F.Cu at (184.4, 97.2)
- added D135: LED_WS2812B, ScottoKeebs_Components:LED_WS2812B, F.Cu at (184.4, 103.9)
- added D136: LED_WS2812B, ScottoKeebs_Components:LED_WS2812B, F.Cu at (192.8, 11.2)
- added D137: LED_WS2812B, ScottoKeebs_Components:LED_WS2812B, F.Cu at (192.8, 17.8)
- added D138: LED_WS2812B, ScottoKeebs_Components:LED_WS2812B, F.Cu at (192.8, 24.4)
- added D139: LED_WS2812B, ScottoKeebs_Components:LED_WS2812B, F.Cu at (192.8, 31.0)
- added D14: Diode, ScottoKeebs_Components:Diode_SOD-123, F.Cu at (132.4, 9.54)
- added D140: LED_WS2812B, ScottoKeebs_Components:LED_WS2812B, F.Cu at (192.8, 37.7)
- added D141: LED_WS2812B, ScottoKeebs_Components:LED_WS2812B, F.Cu at (192.8, 44.3)
- added D142: LED_WS2812B, ScottoKeebs_Components:LED_WS2812B, F.Cu at (192.8, 50.9)
- added D143: LED_WS2812B, ScottoKeebs_Components:LED_WS2812B, F.Cu at (192.8, 57.5)
- added D144: LED_WS2812B, ScottoKeebs_Components:LED_WS2812B, F.Cu at (192.8, 64.1)
- added D145: LED_WS2812B, ScottoKeebs_Components:LED_WS2812B, F.Cu at (192.8, 70.8)
- added D146: LED_WS2812B, ScottoKeebs_Components:LED_WS2812B, F.Cu at (192.8, 77.4)
- added D147: LED_WS2812B, ScottoKeebs_Components:LED_WS2812B, F.Cu at (192.8, 84.0)
- added D148: LED_WS2812B, ScottoKeebs_Components:LED_WS2812B, F.Cu at (192.8, 90.6)
- added D149: LED_WS2812B, ScottoKeebs_Components:LED_WS2812B, F.Cu at (192.8, 97.2)
- added D15: Diode, ScottoKeebs_Components:Diode_SOD-123, F.Cu at (132.4, 12.9)
- added D150: LED_WS2812B, ScottoKeebs_Components:LED_WS2812B, F.Cu at (192.8, 103.9)
- added D151: LED_WS2812B, ScottoKeebs_Components:LED_WS2812B, F.Cu at (201.2, 11.2)
- added D152: LED_WS2812B, ScottoKeebs_Components:LED_WS2812B, F.Cu at (201.2, 17.8)
- added D153: LED_WS2812B, ScottoKeebs_Components:LED_WS2812B, F.Cu at (201.2, 24.4)
- added D154: LED_WS2812B, ScottoKeebs_Components:LED_WS2812B, F.Cu at (201.2, 31.0)
- added D155: LED_WS2812B, ScottoKeebs_Components:LED_WS2812B, F.Cu at (201.2, 37.7)
- added D156: LED_WS2812B, ScottoKeebs_Components:LED_WS2812B, F.Cu at (201.2, 44.3)
- added D157: LED_WS2812B, ScottoKeebs_Components:LED_WS2812B, F.Cu at (201.2, 50.9)
- added D158: LED_WS2812B, ScottoKeebs_Components:LED_WS2812B, F.Cu at (201.2, 57.5)
- added D159: LED_WS2812B, ScottoKeebs_Components:LED_WS2812B, F.Cu at (201.2, 64.1)
- added D16: Diode, ScottoKeebs_Components:Diode_SOD-123, F.Cu at (132.4, 16.2)
- added D160: LED_WS2812B, ScottoKeebs_Components:LED_WS2812B, F.Cu at (201.2, 70.8)
- added D161: LED_WS2812B, ScottoKeebs_Components:LED_WS2812B, F.Cu at (201.2, 77.4)
- added D162: LED_WS2812B, ScottoKeebs_Components:LED_WS2812B, F.Cu at (201.2, 84.0)
- added D163: LED_WS2812B, ScottoKeebs_Components:LED_WS2812B, F.Cu at (201.2, 90.6)
- added D164: LED_WS2812B, ScottoKeebs_Components:LED_WS2812B, F.Cu at (201.2, 97.2)
- added D165: LED_WS2812B, ScottoKeebs_Components:LED_WS2812B, F.Cu at (201.2, 103.9)
- added D166: LED_WS2812B, ScottoKeebs_Components:LED_WS2812B, F.Cu at (209.6, 11.2)
- added D167: LED_WS2812B, ScottoKeebs_Components:LED_WS2812B, F.Cu at (209.6, 17.8)
- added D168: LED_WS2812B, ScottoKeebs_Components:LED_WS2812B, F.Cu at (209.6, 24.4)
- added D169: LED_WS2812B, ScottoKeebs_Components:LED_WS2812B, F.Cu at (209.6, 31.0)
- added D17: Diode, ScottoKeebs_Components:Diode_SOD-123, F.Cu at (132.4, 19.6)
- added D170: LED_WS2812B, ScottoKeebs_Components:LED_WS2812B, F.Cu at (209.6, 37.7)
- added D171: LED_WS2812B, ScottoKeebs_Components:LED_WS2812B, F.Cu at (209.6, 44.3)
- added D172: LED_WS2812B, ScottoKeebs_Components:LED_WS2812B, F.Cu at (209.6, 50.9)
- added D173: LED_WS2812B, ScottoKeebs_Components:LED_WS2812B, F.Cu at (209.6, 57.5)
- added D174: LED_WS2812B, ScottoKeebs_Components:LED_WS2812B, F.Cu at (209.6, 64.1)
- added D175: LED_WS2812B, ScottoKeebs_Components:LED_WS2812B, F.Cu at (209.6, 70.8)
- added D176: LED_WS2812B, ScottoKeebs_Components:LED_WS2812B, F.Cu at (209.6, 77.4)
- added D177: LED_WS2812B, ScottoKeebs_Components:LED_WS2812B, F.Cu at (209.6, 84.0)
- added D178: LED_WS2812B, ScottoKeebs_Components:LED_WS2812B, F.Cu at (209.6, 90.6)
- added D179: LED_WS2812B, ScottoKeebs_Components:LED_WS2812B, F.Cu at (209.6, 97.2)
- added D18: Diode, ScottoKeebs_Components:Diode_SOD-123, F.Cu at (132.4, 22.9)
- added D180: LED_WS2812B, ScottoKeebs_Components:LED_WS2812B, F.Cu at (209.6, 103.9)
- added D181: LED_WS2812B, ScottoKeebs_Components:LED_WS2812B, F.Cu at (218.1, 11.2)
- added D182: LED_WS2812B, ScottoKeebs_Components:LED_WS2812B, F.Cu at (218.1, 17.8)
- added D183: LED_WS2812B, ScottoKeebs_Components:LED_WS2812B, F.Cu at (218.1, 24.4)
- added D184: LED_WS2812B, ScottoKeebs_Components:LED_WS2812B, F.Cu at (218.1, 31.0)
- added D185: LED_WS2812B, ScottoKeebs_Components:LED_WS2812B, F.Cu at (218.1, 37.7)
- added D186: LED_WS2812B, ScottoKeebs_Components:LED_WS2812B, F.Cu at (218.1, 44.3)
- added D187: LED_WS2812B, ScottoKeebs_Components:LED_WS2812B, F.Cu at (218.1, 50.9)
- added D188: LED_WS2812B, ScottoKeebs_Components:LED_WS2812B, F.Cu at (218.1, 57.5)
- added D189: LED_WS2812B, ScottoKeebs_Components:LED_WS2812B, F.Cu at (218.1, 64.1)
- added D19: Diode, ScottoKeebs_Components:Diode_SOD-123, F.Cu at (132.4, 26.3)
- added D190: LED_WS2812B, ScottoKeebs_Components:LED_WS2812B, F.Cu at (218.1, 70.8)
- added D191: LED_WS2812B, ScottoKeebs_Components:LED_WS2812B, F.Cu at (218.1, 77.4)
- added D192: LED_WS2812B, ScottoKeebs_Components:LED_WS2812B, F.Cu at (218.1, 84.0)
- added D193: LED_WS2812B, ScottoKeebs_Components:LED_WS2812B, F.Cu at (218.1, 90.6)
- added D194: LED_WS2812B, ScottoKeebs_Components:LED_WS2812B, F.Cu at (218.1, 97.2)
- added D195: LED_WS2812B, ScottoKeebs_Components:LED_WS2812B, F.Cu at (218.1, 103.9)
- added D196: LED_WS2812B, ScottoKeebs_Components:LED_WS2812B, F.Cu at (226.5, 11.2)
- added D197: LED_WS2812B, ScottoKeebs_Components:LED_WS2812B, F.Cu at (226.5, 17.8)
- added D198: LED_WS2812B, ScottoKeebs_Components:LED_WS2812B, F.Cu at (226.5, 24.4)
- added D199: LED_WS2812B, ScottoKeebs_Components:LED_WS2812B, F.Cu at (226.5, 31.0)
- added D2: Diode, ScottoKeebs_Components:Diode_SOD-123, F.Cu at (126.6, 12.9)
- added D20: Diode, ScottoKeebs_Components:Diode_SOD-123, F.Cu at (132.4, 29.6)
- added D200: LED_WS2812B, ScottoKeebs_Components:LED_WS2812B, F.Cu at (226.5, 37.7)
- added D201: LED_WS2812B, ScottoKeebs_Components:LED_WS2812B, F.Cu at (226.5, 44.3)
- added D202: LED_WS2812B, ScottoKeebs_Components:LED_WS2812B, F.Cu at (226.5, 50.9)
- added D203: LED_WS2812B, ScottoKeebs_Components:LED_WS2812B, F.Cu at (226.5, 57.5)
- added D204: LED_WS2812B, ScottoKeebs_Components:LED_WS2812B, F.Cu at (226.5, 64.1)
- added D205: LED_WS2812B, ScottoKeebs_Components:LED_WS2812B, F.Cu at (226.5, 70.8)
- added D206: LED_WS2812B, ScottoKeebs_Components:LED_WS2812B, F.Cu at (226.5, 77.4)
- added D207: LED_WS2812B, ScottoKeebs_Components:LED_WS2812B, F.Cu at (226.5, 84.0)
- added D208: LED_WS2812B, ScottoKeebs_Components:LED_WS2812B, F.Cu at (226.5, 90.6)
- added D209: LED_WS2812B, ScottoKeebs_Components:LED_WS2812B, F.Cu at (226.5, 97.2)
- added D21: Diode, ScottoKeebs_Components:Diode_SOD-123, F.Cu at (132.4, 33.0)
- added D210: LED_WS2812B, ScottoKeebs_Components:LED_WS2812B, F.Cu at (226.5, 103.9)
- added D211: LED_WS2812B, ScottoKeebs_Components:LED_WS2812B, F.Cu at (234.9, 11.2)
- added D212: LED_WS2812B, ScottoKeebs_Components:LED_WS2812B, F.Cu at (234.9, 17.8)
- added D213: LED_WS2812B, ScottoKeebs_Components:LED_WS2812B, F.Cu at (234.9, 24.4)
- added D214: LED_WS2812B, ScottoKeebs_Components:LED_WS2812B, F.Cu at (234.9, 31.0)
- added D215: LED_WS2812B, ScottoKeebs_Components:LED_WS2812B, F.Cu at (234.9, 37.7)
- added D216: LED_WS2812B, ScottoKeebs_Components:LED_WS2812B, F.Cu at (234.9, 44.3)
- added D217: LED_WS2812B, ScottoKeebs_Components:LED_WS2812B, F.Cu at (234.9, 50.9)
- added D218: LED_WS2812B, ScottoKeebs_Components:LED_WS2812B, F.Cu at (234.9, 57.5)
- added D219: LED_WS2812B, ScottoKeebs_Components:LED_WS2812B, F.Cu at (234.9, 64.1)
- added D22: Diode, ScottoKeebs_Components:Diode_SOD-123, F.Cu at (132.4, 36.3)
- added D220: LED_WS2812B, ScottoKeebs_Components:LED_WS2812B, F.Cu at (234.9, 70.8)
- added D221: LED_WS2812B, ScottoKeebs_Components:LED_WS2812B, F.Cu at (234.9, 77.4)
- added D222: LED_WS2812B, ScottoKeebs_Components:LED_WS2812B, F.Cu at (234.9, 84.0)
- added D223: LED_WS2812B, ScottoKeebs_Components:LED_WS2812B, F.Cu at (234.9, 90.6)
- added D224: LED_WS2812B, ScottoKeebs_Components:LED_WS2812B, F.Cu at (234.9, 97.2)
- added D225: LED_WS2812B, ScottoKeebs_Components:LED_WS2812B, F.Cu at (234.9, 103.9)
- added D226: LED_WS2812B, ScottoKeebs_Components:LED_WS2812B, F.Cu at (243.3, 11.2)
- added D227: LED_WS2812B, ScottoKeebs_Components:LED_WS2812B, F.Cu at (243.3, 17.8)
- added D228: LED_WS2812B, ScottoKeebs_Components:LED_WS2812B, F.Cu at (243.3, 24.4)
- added D229: LED_WS2812B, ScottoKeebs_Components:LED_WS2812B, F.Cu at (243.3, 31.0)
- added D23: Diode, ScottoKeebs_Components:Diode_SOD-123, F.Cu at (132.4, 39.7)
- added D230: LED_WS2812B, ScottoKeebs_Components:LED_WS2812B, F.Cu at (243.3, 37.7)
- added D231: LED_WS2812B, ScottoKeebs_Components:LED_WS2812B, F.Cu at (243.3, 44.3)
- added D232: LED_WS2812B, ScottoKeebs_Components:LED_WS2812B, F.Cu at (243.3, 50.9)
- added D233: LED_WS2812B, ScottoKeebs_Components:LED_WS2812B, F.Cu at (243.3, 57.5)
- added D234: LED_WS2812B, ScottoKeebs_Components:LED_WS2812B, F.Cu at (243.3, 64.1)
- added D235: LED_WS2812B, ScottoKeebs_Components:LED_WS2812B, F.Cu at (243.3, 70.8)
- added D236: LED_WS2812B, ScottoKeebs_Components:LED_WS2812B, F.Cu at (243.3, 77.4)
- added D237: LED_WS2812B, ScottoKeebs_Components:LED_WS2812B, F.Cu at (243.3, 84.0)
- added D238: LED_WS2812B, ScottoKeebs_Components:LED_WS2812B, F.Cu at (243.3, 90.6)
- added D239: LED_WS2812B, ScottoKeebs_Components:LED_WS2812B, F.Cu at (243.3, 97.2)
- added D24: Diode, ScottoKeebs_Components:Diode_SOD-123, F.Cu at (132.4, 43.0)
- added D240: LED_WS2812B, ScottoKeebs_Components:LED_WS2812B, F.Cu at (243.3, 103.9)
- added D241: LED_WS2812B, ScottoKeebs_Components:LED_WS2812B, F.Cu at (251.7, 11.2)
- added D242: LED_WS2812B, ScottoKeebs_Components:LED_WS2812B, F.Cu at (251.7, 17.8)
- added D243: LED_WS2812B, ScottoKeebs_Components:LED_WS2812B, F.Cu at (251.7, 24.4)
- added D244: LED_WS2812B, ScottoKeebs_Components:LED_WS2812B, F.Cu at (251.7, 31.0)
- added D245: LED_WS2812B, ScottoKeebs_Components:LED_WS2812B, F.Cu at (251.7, 37.7)
- added D246: LED_WS2812B, ScottoKeebs_Components:LED_WS2812B, F.Cu at (251.7, 44.3)
- added D247: LED_WS2812B, ScottoKeebs_Components:LED_WS2812B, F.Cu at (251.7, 50.9)
- added D248: LED_WS2812B, ScottoKeebs_Components:LED_WS2812B, F.Cu at (251.7, 57.5)
- added D249: LED_WS2812B, ScottoKeebs_Components:LED_WS2812B, F.Cu at (251.7, 64.1)
- added D25: Diode, ScottoKeebs_Components:Diode_SOD-123, F.Cu at (132.4, 46.4)
- added D26: Diode, ScottoKeebs_Components:Diode_SOD-123, F.Cu at (132.4, 49.7)
- added D27: Diode, ScottoKeebs_Components:Diode_SOD-123, F.Cu at (138.1, 9.54)
- added D28: Diode, ScottoKeebs_Components:Diode_SOD-123, F.Cu at (138.1, 12.9)
- added D29: Diode, ScottoKeebs_Components:Diode_SOD-123, F.Cu at (138.1, 16.2)
- added D3: Diode, ScottoKeebs_Components:Diode_SOD-123, F.Cu at (126.6, 16.2)
- added D30: Diode, ScottoKeebs_Components:Diode_SOD-123, F.Cu at (138.1, 19.6)
- added D31: Diode, ScottoKeebs_Components:Diode_SOD-123, F.Cu at (138.1, 22.9)
- added D32: Diode, ScottoKeebs_Components:Diode_SOD-123, F.Cu at (138.1, 26.3)
- added D33: Diode, ScottoKeebs_Components:Diode_SOD-123, F.Cu at (138.1, 29.6)
- added D34: Diode, ScottoKeebs_Components:Diode_SOD-123, F.Cu at (138.1, 33.0)
- added D35: Diode, ScottoKeebs_Components:Diode_SOD-123, F.Cu at (138.1, 36.3)
- added D36: Diode, ScottoKeebs_Components:Diode_SOD-123, F.Cu at (138.1, 39.7)
- added D37: Diode, ScottoKeebs_Components:Diode_SOD-123, F.Cu at (138.1, 43.0)
- added D38: Diode, ScottoKeebs_Components:Diode_SOD-123, F.Cu at (138.1, 46.4)
- added D39: Diode, ScottoKeebs_Components:Diode_SOD-123, F.Cu at (138.1, 49.7)
- added D4: Diode, ScottoKeebs_Components:Diode_SOD-123, F.Cu at (126.6, 19.6)
- added D40: Diode, ScottoKeebs_Components:Diode_SOD-123, F.Cu at (143.9, 9.54)
- added D41: Diode, ScottoKeebs_Components:Diode_SOD-123, F.Cu at (143.9, 12.9)
- added D42: Diode, ScottoKeebs_Components:Diode_SOD-123, F.Cu at (143.9, 16.2)
- added D43: Diode, ScottoKeebs_Components:Diode_SOD-123, F.Cu at (143.9, 19.6)
- added D44: Diode, ScottoKeebs_Components:Diode_SOD-123, F.Cu at (143.9, 22.9)
- added D45: Diode, ScottoKeebs_Components:Diode_SOD-123, F.Cu at (143.9, 26.3)
- added D46: Diode, ScottoKeebs_Components:Diode_SOD-123, F.Cu at (143.9, 29.6)
- added D47: Diode, ScottoKeebs_Components:Diode_SOD-123, F.Cu at (143.9, 33.0)
- added D48: Diode, ScottoKeebs_Components:Diode_SOD-123, F.Cu at (143.9, 36.3)
- added D49: Diode, ScottoKeebs_Components:Diode_SOD-123, F.Cu at (143.9, 39.7)
- added D5: Diode, ScottoKeebs_Components:Diode_SOD-123, F.Cu at (126.6, 22.9)
- added D50: Diode, ScottoKeebs_Components:Diode_SOD-123, F.Cu at (143.9, 43.0)
- added D51: Diode, ScottoKeebs_Components:Diode_SOD-123, F.Cu at (143.9, 46.4)
- added D52: Diode, ScottoKeebs_Components:Diode_SOD-123, F.Cu at (143.9, 49.7)
- added D53: Diode, ScottoKeebs_Components:Diode_SOD-123, F.Cu at (149.6, 9.54)
- added D54: Diode, ScottoKeebs_Components:Diode_SOD-123, F.Cu at (149.6, 12.9)
- added D55: Diode, ScottoKeebs_Components:Diode_SOD-123, F.Cu at (149.6, 16.2)
- added D56: Diode, ScottoKeebs_Components:Diode_SOD-123, F.Cu at (149.6, 19.6)
- added D57: Diode, ScottoKeebs_Components:Diode_SOD-123, F.Cu at (149.6, 22.9)
- added D58: Diode, ScottoKeebs_Components:Diode_SOD-123, F.Cu at (149.6, 26.3)
- added D59: Diode, ScottoKeebs_Components:Diode_SOD-123, F.Cu at (149.6, 29.6)
- added D6: Diode, ScottoKeebs_Components:Diode_SOD-123, F.Cu at (126.6, 26.3)
- added D60: Diode, ScottoKeebs_Components:Diode_SOD-123, F.Cu at (149.6, 33.0)
- added D61: Diode, ScottoKeebs_Components:Diode_SOD-123, F.Cu at (149.6, 36.3)
- added D62: Diode, ScottoKeebs_Components:Diode_SOD-123, F.Cu at (149.6, 39.7)
- added D63: Diode, ScottoKeebs_Components:Diode_SOD-123, F.Cu at (149.6, 43.0)
- added D64: Diode, ScottoKeebs_Components:Diode_SOD-123, F.Cu at (149.6, 46.4)
- added D65: Diode, ScottoKeebs_Components:Diode_SOD-123, F.Cu at (149.6, 49.7)
- added D66: Diode, ScottoKeebs_Components:Diode_SOD-123, F.Cu at (155.4, 9.54)
- added D67: Diode, ScottoKeebs_Components:Diode_SOD-123, F.Cu at (155.4, 12.9)
- added D68: Diode, ScottoKeebs_Components:Diode_SOD-123, F.Cu at (155.4, 16.2)
- added D69: Diode, ScottoKeebs_Components:Diode_SOD-123, F.Cu at (155.4, 19.6)
- added D7: Diode, ScottoKeebs_Components:Diode_SOD-123, F.Cu at (126.6, 29.6)
- added D70: Diode, ScottoKeebs_Components:Diode_SOD-123, F.Cu at (155.4, 22.9)
- added D71: Diode, ScottoKeebs_Components:Diode_SOD-123, F.Cu at (155.4, 26.3)
- added D72: Diode, ScottoKeebs_Components:Diode_SOD-123, F.Cu at (155.4, 29.6)
- added D73: Diode, ScottoKeebs_Components:Diode_SOD-123, F.Cu at (155.4, 33.0)
- added D74: Diode, ScottoKeebs_Components:Diode_SOD-123, F.Cu at (155.4, 36.3)
- added D75: Diode, ScottoKeebs_Components:Diode_SOD-123, F.Cu at (155.4, 39.7)
- added D76: Diode, ScottoKeebs_Components:Diode_SOD-123, F.Cu at (155.4, 43.0)
- added D77: Diode, ScottoKeebs_Components:Diode_SOD-123, F.Cu at (155.4, 46.4)
- added D78: Diode, ScottoKeebs_Components:Diode_SOD-123, F.Cu at (155.4, 49.7)
- added D79: Diode, ScottoKeebs_Components:Diode_SOD-123, F.Cu at (161.1, 9.54)
- added D8: Diode, ScottoKeebs_Components:Diode_SOD-123, F.Cu at (126.6, 33.0)
- added D80: Diode, ScottoKeebs_Components:Diode_SOD-123, F.Cu at (161.1, 12.9)
- added D81: Diode, ScottoKeebs_Components:Diode_SOD-123, F.Cu at (161.1, 16.2)
- added D82: Diode, ScottoKeebs_Components:Diode_SOD-123, F.Cu at (161.1, 19.6)
- added D83: Diode, ScottoKeebs_Components:Diode_SOD-123, F.Cu at (161.1, 22.9)
- added D84: Diode, ScottoKeebs_Components:Diode_SOD-123, F.Cu at (161.1, 26.3)
- added D85: Diode, ScottoKeebs_Components:Diode_SOD-123, F.Cu at (161.1, 29.6)
- added D86: Diode, ScottoKeebs_Components:Diode_SOD-123, F.Cu at (161.1, 33.0)
- added D87: Diode, ScottoKeebs_Components:Diode_SOD-123, F.Cu at (161.1, 36.3)
- added D88: Diode, ScottoKeebs_Components:Diode_SOD-123, F.Cu at (161.1, 39.7)
- added D89: Diode, ScottoKeebs_Components:Diode_SOD-123, F.Cu at (161.1, 43.0)
- added D9: Diode, ScottoKeebs_Components:Diode_SOD-123, F.Cu at (126.6, 36.3)
- added D90: Diode, ScottoKeebs_Components:Diode_SOD-123, F.Cu at (161.1, 46.4)
- added D91: Diode, ScottoKeebs_Components:Diode_SOD-123, F.Cu at (161.1, 49.7)
- added D92: Diode, ScottoKeebs_Components:Diode_SOD-123, F.Cu at (166.9, 9.54)
- added D93: Diode, ScottoKeebs_Components:Diode_SOD-123, F.Cu at (166.9, 12.9)
- added D94: Diode, ScottoKeebs_Components:Diode_SOD-123, F.Cu at (166.9, 16.2)
- added D95: Diode, ScottoKeebs_Components:Diode_SOD-123, F.Cu at (166.9, 19.6)
- added D96: Diode, ScottoKeebs_Components:Diode_SOD-123, F.Cu at (166.9, 22.9)
- added D97: Diode, ScottoKeebs_Components:Diode_SOD-123, F.Cu at (166.9, 26.3)
- added D98: Diode, ScottoKeebs_Components:Diode_SOD-123, F.Cu at (166.9, 29.6)
- added D99: Diode, ScottoKeebs_Components:Diode_SOD-123, F.Cu at (166.9, 33.0)
- added Delete1: Keyswitch, ScottoKeebs_Hotswap:Hotswap_MX_1.00u, F.Cu at (317.8, 277.2)
- added DownArrow1: Keyswitch, ScottoKeebs_Hotswap:Hotswap_MX_1.00u, F.Cu at (16.2, 15.6)
- added E1: Keyswitch, ScottoKeebs_Hotswap:Hotswap_MX_1.00u, F.Cu at (94.0, 277.2)
- added ESC1: Keyswitch, ScottoKeebs_Hotswap:Hotswap_MX_1.00u, F.Cu at (27.3, 229.6)
- added End1: Keyswitch, ScottoKeebs_Hotswap:Hotswap_MX_1.00u, F.Cu at (336.9, 277.2)
- added Enter1: Keyswitch, ScottoKeebs_Hotswap:Hotswap_MX_1.00u, F.Cu at (16.2, 77.8)
- added F10: Keyswitch, ScottoKeebs_Hotswap:Hotswap_MX_1.00u, F.Cu at (255.9, 229.6)
- added F11: Keyswitch, ScottoKeebs_Hotswap:Hotswap_MX_1.00u, F.Cu at (274.9, 229.6)
- added F12: Keyswitch, ScottoKeebs_Hotswap:Hotswap_MX_1.00u, F.Cu at (294.0, 229.6)
- added F13: Keyswitch, ScottoKeebs_Hotswap:Hotswap_MX_1.00u, F.Cu at (115.4, 296.3)
- added F2: Keyswitch, ScottoKeebs_Hotswap:Hotswap_MX_1.00u, F.Cu at (84.5, 229.6)
- added F3: Keyswitch, ScottoKeebs_Hotswap:Hotswap_MX_1.00u, F.Cu at (103.5, 229.6)
- added F4: Keyswitch, ScottoKeebs_Hotswap:Hotswap_MX_1.00u, F.Cu at (122.6, 229.6)
- added F5: Keyswitch, ScottoKeebs_Hotswap:Hotswap_MX_1.00u, F.Cu at (151.2, 229.6)
- added F6: Keyswitch, ScottoKeebs_Hotswap:Hotswap_MX_1.00u, F.Cu at (170.2, 229.6)
- added F7: Keyswitch, ScottoKeebs_Hotswap:Hotswap_MX_1.00u, F.Cu at (189.2, 229.6)
- added F8: Keyswitch, ScottoKeebs_Hotswap:Hotswap_MX_1.00u, F.Cu at (208.2, 229.6)
- added F9: Keyswitch, ScottoKeebs_Hotswap:Hotswap_MX_1.00u, F.Cu at (236.9, 229.6)
- added Func1: Keyswitch, ScottoKeebs_Hotswap:Hotswap_MX_1.00u, F.Cu at (65.4, 229.6)
- added G1: Keyswitch, ScottoKeebs_Hotswap:Hotswap_MX_1.00u, F.Cu at (134.5, 296.3)
- added H1: Keyswitch, ScottoKeebs_Hotswap:Hotswap_MX_1.00u, F.Cu at (153.5, 296.3)
- added Home1: Keyswitch, ScottoKeebs_Hotswap:Hotswap_MX_1.00u, F.Cu at (336.9, 258.2)
- added I1: Keyswitch, ScottoKeebs_Hotswap:Hotswap_MX_1.00u, F.Cu at (189.3, 277.2)
- added Insert1: Keyswitch, ScottoKeebs_Hotswap:Hotswap_MX_1.00u, F.Cu at (317.8, 258.2)
- added J2: Keyswitch, ScottoKeebs_Hotswap:Hotswap_MX_1.00u, F.Cu at (172.6, 296.3)
- added K1: Keyswitch, ScottoKeebs_Hotswap:Hotswap_MX_1.00u, F.Cu at (191.6, 296.3)
- added L1: Keyswitch, ScottoKeebs_Hotswap:Hotswap_MX_1.00u, F.Cu at (210.7, 296.3)
- added LeftAlt1: Keyswitch, ScottoKeebs_Hotswap:Hotswap_MX_1.00u, F.Cu at (49.4, 46.7)
- added LeftArrow1: Keyswitch, ScottoKeebs_Hotswap:Hotswap_MX_1.00u, F.Cu at (49.4, 62.3)
- added LeftControl1: Keyswitch, ScottoKeebs_Hotswap:Hotswap_MX_1.00u, F.Cu at (49.4, 77.8)
- added LeftWin1: Keyswitch, ScottoKeebs_Hotswap:Hotswap_MX_1.00u, F.Cu at (49.4, 93.4)
- added M1: Keyswitch, ScottoKeebs_Hotswap:Hotswap_MX_1.00u, F.Cu at (49.4, 108.9)
- added Menu1: Keyswitch, ScottoKeebs_Hotswap:Hotswap_MX_1.00u, F.Cu at (49.4, 124.5)
- added N1: Keyswitch, ScottoKeebs_Hotswap:Hotswap_MX_1.00u, F.Cu at (49.4, 140.0)
- added Num*1: Keyswitch, ScottoKeebs_Hotswap:Hotswap_MX_1.00u, F.Cu at (415.5, 258.2)
- added Num-1: Keyswitch, ScottoKeebs_Hotswap:Hotswap_MX_1.00u, F.Cu at (434.5, 258.2)
- added Num.1: Keyswitch, ScottoKeebs_Hotswap:Hotswap_MX_1.00u, F.Cu at (66.1, 171.1)
- added Num/1: Keyswitch, ScottoKeebs_Hotswap:Hotswap_MX_1.00u, F.Cu at (396.4, 258.2)
- added Num0: Keyswitch, ScottoKeebs_Hotswap:Hotswap_MX_1.00u, F.Cu at (49.4, 155.6)
- added Num1: Keyswitch, ScottoKeebs_Hotswap:Hotswap_MX_1.00u, F.Cu at (49.4, 171.1)
- added Num10: Keyswitch, ScottoKeebs_Hotswap:Hotswap_MX_1.00u, F.Cu at (66.1, 124.5)
- added Num2: Keyswitch, ScottoKeebs_Hotswap:Hotswap_MX_1.00u, F.Cu at (49.4, 186.7)
- added Num3: Keyswitch, ScottoKeebs_Hotswap:Hotswap_MX_1.00u, F.Cu at (66.1, 15.6)
- added Num4: Keyswitch, ScottoKeebs_Hotswap:Hotswap_MX_1.00u, F.Cu at (66.1, 31.2)
- added Num5: Keyswitch, ScottoKeebs_Hotswap:Hotswap_MX_1.00u, F.Cu at (66.1, 46.7)
- added Num6: Keyswitch, ScottoKeebs_Hotswap:Hotswap_MX_1.00u, F.Cu at (66.1, 62.3)
- added Num7: Keyswitch, ScottoKeebs_Hotswap:Hotswap_MX_1.00u, F.Cu at (66.1, 77.8)
- added Num8: Keyswitch, ScottoKeebs_Hotswap:Hotswap_MX_1.00u, F.Cu at (66.1, 93.4)
- added Num9: Keyswitch, ScottoKeebs_Hotswap:Hotswap_MX_1.00u, F.Cu at (66.1, 108.9)
- added NumEnter1: Keyswitch, ScottoKeebs_Hotswap:Hotswap_MX_1.00u, F.Cu at (82.7, 15.6)
- added NumLock1: Keyswitch, ScottoKeebs_Hotswap:Hotswap_MX_1.00u, F.Cu at (377.4, 258.2)
- added O1: Keyswitch, ScottoKeebs_Hotswap:Hotswap_MX_1.00u, F.Cu at (208.3, 277.2)
- added P1: Keyswitch, ScottoKeebs_Hotswap:Hotswap_MX_1.00u, F.Cu at (227.4, 277.2)
- added PauseBreak1: Keyswitch, ScottoKeebs_Hotswap:Hotswap_MX_1.00u, F.Cu at (355.9, 229.6)
- added PgDn1: Keyswitch, ScottoKeebs_Hotswap:Hotswap_MX_1.00u, F.Cu at (355.9, 277.2)
- added PgUp1: Keyswitch, ScottoKeebs_Hotswap:Hotswap_MX_1.00u, F.Cu at (355.9, 258.2)
- added PrtSc1: Keyswitch, ScottoKeebs_Hotswap:Hotswap_MX_1.00u, F.Cu at (317.8, 229.6)
- added Q1: Keyswitch, ScottoKeebs_Hotswap:Hotswap_MX_1.00u, F.Cu at (55.9, 277.2)
- added R4: Keyswitch, ScottoKeebs_Hotswap:Hotswap_MX_1.00u, F.Cu at (113.1, 277.2)
- added RightAlt1: Keyswitch, ScottoKeebs_Hotswap:Hotswap_MX_1.00u, F.Cu at (82.7, 171.1)
- added RightArrow1: Keyswitch, ScottoKeebs_Hotswap:Hotswap_MX_1.00u, F.Cu at (82.7, 186.7)
- added RightControl1: Keyswitch, ScottoKeebs_Hotswap:Hotswap_MX_1.00u, F.Cu at (99.3, 15.6)
- added RightWin1: Keyswitch, ScottoKeebs_Hotswap:Hotswap_MX_1.00u, F.Cu at (99.3, 31.2)
- added S1: Keyswitch, ScottoKeebs_Hotswap:Hotswap_MX_1.00u, F.Cu at (77.3, 296.3)
- added ScrollLock1: Keyswitch, ScottoKeebs_Hotswap:Hotswap_MX_1.00u, F.Cu at (336.9, 229.6)
- added Shift1: Keyswitch, ScottoKeebs_Hotswap:Hotswap_MX_1.00u, F.Cu at (99.3, 77.8)
- added Shift2: Keyswitch, ScottoKeebs_Hotswap:Hotswap_MX_1.00u, F.Cu at (99.3, 93.4)
- added Space1: Keyswitch, ScottoKeebs_Hotswap:Hotswap_MX_1.00u, F.Cu at (99.3, 108.9)
- added T1: Keyswitch, ScottoKeebs_Hotswap:Hotswap_MX_1.00u, F.Cu at (132.1, 277.2)
- added Tab1: Keyswitch, ScottoKeebs_Hotswap:Hotswap_MX_1.00u, F.Cu at (32.1, 277.2)
- added Tilde1: Keyswitch, ScottoKeebs_Hotswap:Hotswap_MX_1.00u, F.Cu at (27.3, 258.2)
- added U2: Keyswitch, ScottoKeebs_Hotswap:Hotswap_MX_1.00u, F.Cu at (170.2, 277.2)
- added UpArrow1: Keyswitch, ScottoKeebs_Hotswap:Hotswap_MX_1.00u, F.Cu at (136.6, 196.2)
- added V1: Keyswitch, ScottoKeebs_Hotswap:Hotswap_MX_1.00u, F.Cu at (116.0, 15.6)
- added W1: Keyswitch, ScottoKeebs_Hotswap:Hotswap_MX_1.00u, F.Cu at (75.0, 277.2)
- added X1: Keyswitch, ScottoKeebs_Hotswap:Hotswap_MX_1.00u, F.Cu at (116.0, 46.7)
- added Y1: Keyswitch, ScottoKeebs_Hotswap:Hotswap_MX_1.00u, F.Cu at (151.2, 277.2)
- added Z1: Keyswitch, ScottoKeebs_Hotswap:Hotswap_MX_1.00u, F.Cu at (116.0, 77.8)
- added \1: Keyswitch, ScottoKeebs_Hotswap:Hotswap_MX_1.00u, F.Cu at (289.3, 277.2)
- added {1: Keyswitch, ScottoKeebs_Hotswap:Hotswap_MX_1.00u, F.Cu at (246.4, 277.2)
- added }1: Keyswitch, ScottoKeebs_Hotswap:Hotswap_MX_1.00u, F.Cu at (265.5, 277.2)
Connections:
- U1 pad 10: /A0 -> Col10
- U1 pad 11: /A1 -> Col11
- U1 pad 12: /A2 -> Col12
- U1 pad 13: /A3 -> Col13
- U1 pad 14: /A4 -> Col14
- U1 pad 15: /A5 -> Col15
- U1 pad 16: /A6 -> Col16
- U1 pad 17: /A7 -> Col17
- U1 pad 18: /B0 -> Row0
- U1 pad 19: /B1 -> Row1
- U1 pad 20: /B2 -> Row2
- U1 pad 21: /B10 -> Col4
- U1 pad 22: /B11 -> Col5
- U1 pad 25: /B12 -> Col6
- U1 pad 26: /B13 -> Col7
- U1 pad 27: /B14 -> Col8
- U1 pad 28: /B15 -> Col9
- U1 pad 29: /A8 -> Col18
- U1 pad 30: /A9 -> Col19
- U1 pad 31: /A10 -> Col20
- U1 pad 38: /A15 -> LEDIN
- U1 pad 39: /B3 -> Row3
- U1 pad 40: /B4 -> Row4
- U1 pad 41: /B5 -> Row5
- U1 pad 42: /B6 -> Col0
- U1 pad 43: /B7 -> Col1
- U1 pad 45: /B8 -> Col2
- U1 pad 46: /B9 -> Col3
Routing:
- removed copper zone on In1.Cu, net GND
- removed copper zone on In2.Cu, net GND
