File: PCB/Full Keyboard.kicad_pcb (KiCad board)
At the start: 4 copper layers, 38.1 x 57.2 mm, 378 parts, among them J1 USB_C, J2 Keyswitch, K1 Keyswitch, M1 Keyswitch, P1 Keyswitch, Q1 Keyswitch, SW1 SW_Push, T1 Keyswitch, U1 STM32F072CBT6, U2 Keyswitch, U3 XC6206, U4 USBLC6-2SC6, X1 Keyswitch, Y1 Keyswitch

Commit message: PCB Design
Parts:
- removed REF** (x6): MX_1.00u_PG151101S11, ScottoKeebs_Scotto:MX_Hotswap_1.00u
- Backspace1, Num0: footprint ScottoKeebs_Hotswap:Hotswap_MX_1.00u -> ScottoKeebs_Hotswap:Hotswap_MX_2.00u
- CapsLock1: footprint ScottoKeebs_Hotswap:Hotswap_MX_1.00u -> ScottoKeebs_Hotswap:Hotswap_MX_1.75u
- D1, D10, D100, D101, D102, D103, D104, D11, D12, D13, D14, D15, D16, D17, D18, D19, D2, D20, D21, D22, D23, D24, D25, D26, D27, D28, D29, D3, D30, D31, D32, D33, D34, D35, D36, D37, D38, D39, D4, D40, D41, D42, D43, D44, D45, D46, D47, D48, D49, D5, D50, D51, D52, D53, D54, D55, D56, D57, D58, D59, D6, D60, D61, D62, D63, D64, D65, D66, D67, D68, D69, D7, D70, D71, D72, D73, D74, D75, D76, D77, D78, D79, D8, D80, D81, D82, D83, D84, D85, D86, D87, D88, D89, D9, D90, D91, D92, D93, D94, D95, D96, D97, D98, D99: moved to B.Cu
- Enter1, Shift1: footprint ScottoKeebs_Hotswap:Hotswap_MX_1.00u -> ScottoKeebs_Hotswap:Hotswap_MX_2.25u
- LeftAlt1, LeftControl1, LeftWin1, Menu1, RightAlt1, RightControl1, RightWin1: footprint ScottoKeebs_Hotswap:Hotswap_MX_1.00u -> ScottoKeebs_Hotswap:Hotswap_MX_1.25u
- Num+1: renamed from Num10; footprint ScottoKeebs_Hotswap:Hotswap_MX_1.00u -> ScottoKeebs_Hotswap:Hotswap_MX_2.00u_90deg
- NumEnter1: footprint ScottoKeebs_Hotswap:Hotswap_MX_1.00u -> ScottoKeebs_Hotswap:Hotswap_MX_2.00u_90deg
- RightShift1: renamed from Shift2; footprint ScottoKeebs_Hotswap:Hotswap_MX_1.00u -> ScottoKeebs_Hotswap:Hotswap_MX_2.75u
- Space1: footprint ScottoKeebs_Hotswap:Hotswap_MX_1.00u -> ScottoKeebs_Hotswap:Hotswap_MX_6.25u
- Tab1, \1: footprint ScottoKeebs_Hotswap:Hotswap_MX_1.00u -> ScottoKeebs_Hotswap:Hotswap_MX_1.50u
- moved NumEnter1 537.5 mm to (522.3, 324.8)
- moved Num3 530.0 mm to (503.3, 315.3)
- moved DownArrow1 516.3 mm to (422.3, 334.4)
- moved Num6 495.9 mm to (503.3, 296.3)
- moved Num5 486.9 mm to (484.2, 296.3)
- moved Num+1 484.2 mm to (522.3, 286.7)
- moved Num4 479.1 mm to (465.2, 296.3)
- moved Num9 468.5 mm to (503.3, 277.2)
- moved Num.1 466.7 mm to (503.3, 334.4)
- moved Num0 461.3 mm to (474.7, 334.4)
- moved D58 460.4 mm to (531.7, 283.2), turned to 90 degrees
- moved D91 459.6 mm to (531.8, 321.4), turned to 90 degrees
- moved Num8 456.8 mm to (484.2, 277.2)
- moved Num2 453.4 mm to (484.2, 315.3)
- moved D37 446.7 mm to (531.5, 254.7), turned to 90 degrees
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Connections:
- U1 pad 10: Col10 -> (no net)
- U1 pad 11: Col11 -> (no net)
- U1 pad 12: Col12 -> (no net)
- U1 pad 13: Col13 -> (no net)
- U1 pad 14: Col14 -> (no net)
- U1 pad 15: Col15 -> (no net)
- U1 pad 16: Col16 -> (no net)
- U1 pad 17: Col17 -> (no net)
- U1 pad 18: Row0 -> (no net)
- U1 pad 19: Row1 -> (no net)
- U1 pad 20: Row2 -> (no net)
- U1 pad 21: Col4 -> (no net)
- U1 pad 22: Col5 -> (no net)
- U1 pad 25: Col6 -> (no net)
- U1 pad 26: Col7 -> (no net)
- U1 pad 27: Col8 -> (no net)
- U1 pad 28: Col9 -> (no net)
- U1 pad 29: Col18 -> (no net)
- U1 pad 30: Col19 -> (no net)
- U1 pad 31: Col20 -> (no net)
- U1 pad 38: LEDIN -> (no net)
- U1 pad 39: Row3 -> (no net)
- U1 pad 40: Row4 -> (no net)
- U1 pad 41: Row5 -> (no net)
- U1 pad 42: Col0 -> (no net)
- U1 pad 43: Col1 -> (no net)
- U1 pad 45: Col2 -> (no net)
- U1 pad 46: Col3 -> (no net)
Routing:
- added copper zone on In1.Cu, net GND
- added copper zone on In2.Cu, net GND
