File: PCB/Full Keyboard.kicad_sch (KiCad schematic)
At the start: 228 parts, among them J1 USB_C, J2 Keyswitch, K1 Keyswitch, M1 Keyswitch, P1 Keyswitch, Q1 Keyswitch, SW1 SW_Push, T1 Keyswitch, U1 STM32F072CBT6, U2 Keyswitch, U3 XC6206, U4 USBLC6-2SC6, X1 Keyswitch, Y1 Keyswitch

Commit message: PCB Design
Parts:
- Backspace1, Num0: footprint ScottoKeebs_Hotswap:Hotswap_MX_1.00u -> ScottoKeebs_Hotswap:Hotswap_MX_2.00u
- CapsLock1: footprint ScottoKeebs_Hotswap:Hotswap_MX_1.00u -> ScottoKeebs_Hotswap:Hotswap_MX_1.75u
- Enter1, Shift1: footprint ScottoKeebs_Hotswap:Hotswap_MX_1.00u -> ScottoKeebs_Hotswap:Hotswap_MX_2.25u
- LeftAlt1, LeftControl1, LeftWin1, Menu1, RightAlt1, RightControl1, RightWin1: footprint ScottoKeebs_Hotswap:Hotswap_MX_1.00u -> ScottoKeebs_Hotswap:Hotswap_MX_1.25u
- Num+1: renamed from Num10; footprint ScottoKeebs_Hotswap:Hotswap_MX_1.00u -> ScottoKeebs_Hotswap:Hotswap_MX_2.00u_90deg
- NumEnter1: footprint ScottoKeebs_Hotswap:Hotswap_MX_1.00u -> ScottoKeebs_Hotswap:Hotswap_MX_2.00u_90deg
- RightShift1: renamed from Shift2; footprint ScottoKeebs_Hotswap:Hotswap_MX_1.00u -> ScottoKeebs_Hotswap:Hotswap_MX_2.75u
- Space1: footprint ScottoKeebs_Hotswap:Hotswap_MX_1.00u -> ScottoKeebs_Hotswap:Hotswap_MX_6.25u
- Tab1, \1: footprint ScottoKeebs_Hotswap:Hotswap_MX_1.00u -> ScottoKeebs_Hotswap:Hotswap_MX_1.50u
Connections:
- net A15 renamed LEDIN
Changed lines of the file:
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@@
 	(wire
 		(pts
-			(xy 77.47 210.82) (xy 72.39 210.82)
+			(xy 83.82 210.82) (xy 72.39 210.82)
 		)
 		(stroke
@@
 		)
 	)
+	(global_label "LEDIN"
+		(shape input)
+		(at 83.82 210.82 0)
+		(fields_autoplaced yes)
+		(effects
+			(font
+				(size 1.27 1.27)
+			)
+			(justify left)
+		)
+		(property "Intersheetrefs" "${INTERSHEET_REFS}"
+			(at 92.1876 210.82 0)
+			(effects
+				(font
+					(size 1.27 1.27)
+				)
+				(justify left)
+				(hide yes)
+			)
+		)
+	)
 	(global_label "Row0"
 		(shape input)
@@
 			)
 		)
-		(property "Footprint" "ScottoKeebs_Hotswap:Hotswap_MX_1.00u"
+		(property "Footprint" "ScottoKeebs_Hotswap:Hotswap_MX_2.00u_90deg"
 			(at 396.24 142.24 0)
 			(effects
@@
 			)
 		)
-		(property "Footprint" "ScottoKeebs_Hotswap:Hotswap_MX_1.00u"
+		(property "Footprint" "ScottoKeebs_Hotswap:Hotswap_MX_1.50u"
 			(at 307.34 104.14 0)
 			(effects
@@
 			)
 		)
-		(property "Footprint" "ScottoKeebs_Hotswap:Hotswap_MX_1.00u"
+		(property "Footprint" "ScottoKeebs_Hotswap:Hotswap_MX_1.25u"
 			(at 142.24 161.29 0)
 			(effects
@@
 			)
 		)
-		(property "Footprint" "ScottoKeebs_Hotswap:Hotswap_MX_1.00u"
+		(property "Footprint" "ScottoKeebs_Hotswap:Hotswap_MX_2.00u"
 			(at 358.14 161.29 0)
 			(effects
@@
 			)
 		)
-		(property "Footprint" "ScottoKeebs_Hotswap:Hotswap_MX_1.00u"
+		(property "Footprint" "ScottoKeebs_Hotswap:Hotswap_MX_1.25u"
 			(at 269.24 161.29 0)
 			(effects
@@
 			)
 		)
-		(property "Footprint" "ScottoKeebs_Hotswap:Hotswap_MX_1.00u"
+		(property "Footprint" "ScottoKeebs_Hotswap:Hotswap_MX_6.25u"
 			(at 205.74 161.29 0)
 			(effects
@@
 			)
 		)
-		(property "Footprint" "ScottoKeebs_Hotswap:Hotswap_MX_1.00u"
+		(property "Footprint" "ScottoKeebs_Hotswap:Hotswap_MX_1.50u"
 			(at 142.24 104.14 0)
 			(effects
@@
 			)
 		)
-		(property "Footprint" "ScottoKeebs_Hotswap:Hotswap_MX_1.00u"
+		(property "Footprint" "ScottoKeebs_Hotswap:Hotswap_MX_1.25u"
 			(at 307.34 161.29 0)
 			(effects
@@
 			)
 		)
-		(property "Footprint" "ScottoKeebs_Hotswap:Hotswap_MX_1.00u"
+		(property "Footprint" "ScottoKeebs_Hotswap:Hotswap_MX_2.25u"
 			(at 294.64 123.19 0)
 			(effects
@@
 			)
 		)
-		(property "Footprint" "ScottoKeebs_Hotswap:Hotswap_MX_1.00u"
+		(property "Footprint" "ScottoKeebs_Hotswap:Hotswap_MX_1.25u"
 			(at 154.94 161.29 0)
 			(effects
@@
 			)
 		)
-		(property "Footprint" "ScottoKeebs_Hotswap:Hotswap_MX_1.00u"
+		(property "Footprint" "ScottoKeebs_Hotswap:Hotswap_MX_1.75u"
 			(at 142.24 123.19 0)
 			(effects
@@
 			)
 		)
-		(property "Footprint" "ScottoKeebs_Hotswap:Hotswap_MX_1.00u"
+		(property "Footprint" "ScottoKeebs_Hotswap:Hotswap_MX_1.25u"
 			(at 256.54 161.29 0)
 			(effects
@@
 			)
 		)
-		(property "Footprint" "ScottoKeebs_Hotswap:Hotswap_MX_1.00u"
+		(property "Footprint" "ScottoKeebs_Hotswap:Hotswap_MX_1.25u"
 			(at 167.64 161.29 0)
 			(effects
@@
 		(dnp no)
 		(fields_autoplaced yes)
-		(property "Reference" "Shift2"
+		(property "Reference" "RightShift1"
 			(at 281.94 134.62 0)
 			(effects
@@
 			)
 		)
-		(property "Footprint" "ScottoKeebs_Hotswap:Hotswap_MX_1.00u"
+		(property "Footprint" "ScottoKeebs_Hotswap:Hotswap_MX_2.75u"
 			(at 281.94 142.24 0)
 			(effects
@@
 			(project "Full Keyboard"
 				(path "/92054fa3-5ad0-458e-bd73-acbcf8d11243"
-					(reference "Shift2")
+					(reference "RightShift1")
 					(unit 1)
 				)
@@
 			)
 		)
-		(property "Footprint" "ScottoKeebs_Hotswap:Hotswap_MX_1.00u"
+		(property "Footprint" "ScottoKeebs_Hotswap:Hotswap_MX_1.25u"
 			(at 281.94 161.29 0)
 			(effects
@@
 			)
 		)
-		(property "Footprint" "ScottoKeebs_Hotswap:Hotswap_MX_1.00u"
+		(property "Footprint" "ScottoKeebs_Hotswap:Hotswap_MX_2.00u"
 			(at 307.34 85.09 0)
 			(effects
@@
 			)
 		)
-		(property "Footprint" "ScottoKeebs_Hotswap:Hotswap_MX_1.00u"
+		(property "Footprint" "ScottoKeebs_Hotswap:Hotswap_MX_2.25u"
 			(at 142.24 142.24 0)
 			(effects
@@
 		(dnp no)
 		(fields_autoplaced yes)
-		(property "Reference" "Num10"
+		(property "Reference" "Num+1"
 			(at 396.24 96.52 0)
 			(effects
@@
 			)
 		)
-		(property "Footprint" "ScottoKeebs_Hotswap:Hotswap_MX_1.00u"
+		(property "Footprint" "ScottoKeebs_Hotswap:Hotswap_MX_2.00u_90deg"
 			(at 396.24 104.14 0)
 			(effects
@@
 			(project "Full Keyboard"
 				(path "/92054fa3-5ad0-458e-bd73-acbcf8d11243"
-					(reference "Num10")
+					(reference "Num+1")
 					(unit 1)
 				)

Commit message: update
Connections:
- net A13 is gone; now on net Row5: U1.34 (PA13)
- net A14 is gone; now on net Row4: U1.37 (PA14)
- net C13 is gone; now on net Col15: U1.2 (PC13)
- net C14 is gone; now on net Col14: U1.3 (PC14)
- net C15 is gone; now on net Col13: U1.4 (PC15)
- net F0 is gone; now on net Col12: U1.5 (PF0)
- net F1 is gone; now on net Col11: U1.6 (PF1)
- net LEDIN is gone; now on net Row3: U1.38 (PA15)
- net Col0: now also U1.25 (PB12); no longer U1.42 (PB6)
- net Col1: now also U1.22 (PB11); no longer U1.43 (PB7)
- net Col10: now also U1.13 (PA3); no longer U1.10 (PA0)
- net Col11: no longer U1.11 (PA1)
- net Col12: no longer U1.12 (PA2)
- net Col13: no longer U1.13 (PA3)
- net Col14: no longer U1.14 (PA4)
- net Col15: no longer U1.15 (PA5)
- net Col16: now also U1.46 (PB9); no longer U1.16 (PA6)
- net Col17: now also U1.45 (PB8); no longer U1.17 (PA7)
- net Col18: now also U1.43 (PB7); no longer U1.29 (PA8)
- net Col19: now also U1.42 (PB6); no longer U1.30 (PA9)
- net Col2: now also U1.21 (PB10); no longer U1.45 (PB8)
- net Col20: now also U1.41 (PB5); no longer U1.31 (PA10)
- net Col3: now also U1.20 (PB2); no longer U1.46 (PB9)
- net Col4: now also U1.19 (PB1); no longer U1.21 (PB10)
- net Col5: now also U1.18 (PB0); no longer U1.22 (PB11)
- net Col6: now also U1.17 (PA7); no longer U1.25 (PB12)
- net Col7: now also U1.16 (PA6); no longer U1.26 (PB13)
- net Col8: now also U1.15 (PA5); no longer U1.27 (PB14)
- net Col9: now also U1.14 (PA4); no longer U1.28 (PB15)
- net Row0: now also U1.29 (PA8); no longer U1.18 (PB0)
- net Row1: now also U1.40 (PB4); no longer U1.19 (PB1)
- net Row2: now also U1.39 (PB3); no longer U1.20 (PB2)
- net Row3: no longer U1.39 (PB3)
- net Row4: no longer U1.40 (PB4)
- net Row5: no longer U1.41 (PB5)
- new net A0: U1.10 (PA0)
- new net A1: U1.11 (PA1)
- new net A10: U1.31 (PA10)
- new net A2: U1.12 (PA2)
- new net A9: U1.30 (PA9)
- new net B13: U1.26 (PB13)
- new net B14: U1.27 (PB14)
- new net B15: U1.28 (PB15)

Commit message: push
Parts:
- removed C8, C9: 1uF, ScottoKeebs_Components:Capacitor_0402, symbol Device:C_Small
- removed F1: 500mA, ScottoKeebs_Components:Fuse_0603, symbol Device:Fuse_Small
- removed J1: USB_C, ScottoKeebs_Components:USB_C_HRO_TYPE-C-31-M-12, symbol Connector:USB_C_Receptacle_USB2.0_14P
- removed R2, R3: 5.1k, ScottoKeebs_Components:Resistor_0402, symbol Device:R_Small
- removed U3: XC6206, ScottoKeebs_Components:Voltage_SOT-23, symbol Regulator_Linear:XC6206PxxxMR
- removed U4: USBLC6-2SC6, ScottoKeebs_Components:ESD_SOT-23-6, symbol Power_Protection:USBLC6-2SC6
- added J3: Conn_01x04_Pin, Connector_JST:JST_EH_B4B-EH-A_1x04_P2.50mm_Vertical, symbol Connector:Conn_01x04_Pin
Connections:
- net +3.3V: now also J3.1 (Pin_1)
- net GND: now also J3.4 (Pin_4)
- net MCU_D+: now also J3.2 (Pin_2)
- net MCU_D-: now also J3.3 (Pin_3)
Other:
- note removed: "Connector"
- note removed: "ESD Protection"
- note removed: "USB-C"
- note removed: "Voltage Step Down"

Commit message: push
Parts:
- "-"1, "0"1, "1, "1"1, "2"1, "3"1, "4"1, "5"1, "6"1, "7"1, "8"1, "9"1, "="1, "?"1, ;1, <1, >1, A1, B1, C1, D105, Delete1, DownArrow1, E1, ESC1, End1, F10, F11, F12, F13, F2, F3, F4, F5, F6, F7, F8, F9, Func1, G1, H1, Home1, I1, Insert1, J2, K1, L1, LeftArrow1, M1, N1, Num*1, Num-1, Num.1, Num/1, Num1, Num2, Num3, Num4, Num5, Num6, Num7, Num8, Num9, NumLock1, O1, P1, PauseBreak1, PgDn1, PgUp1, PrtSc1, Q1, R4, RightArrow1, S1, ScrollLock1, T1, Tilde1, U2, UpArrow1, V1, W1, X1, Y1, Z1, {1, }1: footprint ScottoKeebs_Hotswap:Hotswap_MX_1.00u -> ScottoKeebs_MX:MX_PCB_1.00u
- Backspace1: footprint ScottoKeebs_Hotswap:Hotswap_MX_2.00u -> ScottoKeebs_MX:MX_PCB_1.00u
- CapsLock1: footprint ScottoKeebs_Hotswap:Hotswap_MX_1.75u -> ScottoKeebs_MX:MX_PCB_1.75u
- Enter1, Shift1: footprint ScottoKeebs_Hotswap:Hotswap_MX_2.25u -> ScottoKeebs_MX:MX_PCB_2.25u
- LeftAlt1, LeftControl1, LeftWin1, Menu1, RightAlt1, RightControl1, RightWin1: footprint ScottoKeebs_Hotswap:Hotswap_MX_1.25u -> ScottoKeebs_MX:MX_PCB_1.25u
- Num+1, NumEnter1: footprint ScottoKeebs_Hotswap:Hotswap_MX_2.00u_90deg -> ScottoKeebs_MX:MX_PCB_2.00u_90deg
- Num0: footprint ScottoKeebs_Hotswap:Hotswap_MX_2.00u -> ScottoKeebs_MX:MX_PCB_2.00u
- RightShift1: footprint ScottoKeebs_Hotswap:Hotswap_MX_2.75u -> ScottoKeebs_MX:MX_PCB_2.75u
- Space1: footprint ScottoKeebs_Hotswap:Hotswap_MX_6.25u -> ScottoKeebs_MX:MX_Plate_6.25u
- Tab1, \1: footprint ScottoKeebs_Hotswap:Hotswap_MX_1.50u -> ScottoKeebs_MX:MX_PCB_1.50u
Other:
- removed sheet LEDs
